Commit message: world and model creation working properly

File: urdf/epsonvt6.urdf (robot description, URDF)
Before this commit: robot epsonvt6, 7 links, 6 joints
Links:
- link base_link: geometry collision mesh filename=file:///home/gman/ros2_ws/install/robot_arm_6axis/share/rob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; visual mesh filename=file:///home/gman/ros2_ws/install/robot_arm_6axis/share/rob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
- link finger_link: geometry collision mesh filename=file:///home/gman/ros2_ws/install/robot_arm_6axis/share/rob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; visual mesh filename=file:///home/gman/ros2_ws/install/robot_arm_6axis/share/rob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
- link hand_link: geometry collision mesh filename=file:///home/gman/ros2_ws/install/robot_arm_6axis/share/rob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; visual mesh filename=file:///home/gman/ros2_ws/install/robot_arm_6axis/share/rob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
- link swivel_arm_link: geometry collision mesh filename=file:///home/gman/ros2_ws/install/robot_arm_6axis/share/rob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; visual mesh filename=file:///home/gman/ros2_ws/install/robot_arm_6axis/share/rob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
- link swivel_link: geometry collision mesh filename=file:///home/gman/ros2_ws/install/robot_arm_6axis/share/rob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; visual mesh filename=file:///home/gman/ros2_ws/install/robot_arm_6axis/share/rob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
- link tip_link: geometry collision mesh filename=file:///home/gman/ros2_ws/install/robot_arm_6axis/share/rob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; visual mesh filename=file:///home/gman/ros2_ws/install/robot_arm_6axis/share/rob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
- link wrist_link: geometry collision mesh filename=file:///home/gman/ros2_ws/install/robot_arm_6axis/share/rob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; visual mesh filename=file:///home/gman/ros2_ws/install/robot_arm_6axis/share/rob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

File: urdf/epsonvt6_core.xacro (robot description, xacro)
@@ -26,5 +26,5 @@
       <geometry>
         <mesh
-          filename="package://robot_arm_6axis/meshes/base_link.STL" />
+          filename="file://$(find robot_arm_6axis)/meshes/base_link.STL" /> <!-- package://robot_arm_6axis/meshes/base_link.STL"-->
       </geometry>
       <material
@@ -40,5 +40,5 @@
       <geometry>
         <mesh
-          filename="package://robot_arm_6axis/meshes/base_link.STL" />
+          filename="file://$(find robot_arm_6axis)/meshes/base_link.STL" />
       </geometry>
     </collision>
@@ -66,5 +66,5 @@
       <geometry>
         <mesh
-          filename="package://robot_arm_6axis/meshes/swivel_link.STL" />
+          filename="file://$(find robot_arm_6axis)/meshes/swivel_link.STL" />
       </geometry>
       <material
@@ -80,5 +80,5 @@
       <geometry>
         <mesh
-          filename="package://robot_arm_6axis/meshes/swivel_link.STL" />
+          filename="file://$(find robot_arm_6axis)/meshes/swivel_link.STL" />
       </geometry>
     </collision>
@@ -119,19 +119,19 @@
       <geometry>
         <mesh
-          filename="package://robot_arm_6axis/meshes/swivel_arm_link.STL" />
-      </geometry>
-      <material
-        name="">
-        <color
-          rgba="0.792156862745098 0.819607843137255 0.933333333333333 1" />
-      </material>
-    </visual>
-    <collision>
-      <origin
-        xyz="0 0 0"
-        rpy="0 0 0" />
-      <geometry>
-        <mesh
-          filename="package://robot_arm_6axis/meshes/swivel_arm_link.STL" />
+          filename="file://$(find robot_arm_6axis)/meshes/swivel_arm_link.STL" />
+      </geometry>
+      <material
+        name="">
+        <color
+          rgba="0.792156862745098 0.819607843137255 0.933333333333333 1" />
+      </material>
+    </visual>
+    <collision>
+      <origin
+        xyz="0 0 0"
+        rpy="0 0 0" />
+      <geometry>
+        <mesh
+          filename="file://$(find robot_arm_6axis)/meshes/swivel_arm_link.STL" />
       </geometry>
     </collision>
@@ -172,19 +172,19 @@
       <geometry>
         <mesh
-          filename="package://robot_arm_6axis/meshes/wrist_link.STL" />
-      </geometry>
-      <material
-        name="">
-        <color
-          rgba="0.792156862745098 0.819607843137255 0.933333333333333 1" />
-      </material>
-    </visual>
-    <collision>
-      <origin
-        xyz="0 0 0"
-        rpy="0 0 0" />
-      <geometry>
-        <mesh
-          filename="package://robot_arm_6axis/meshes/wrist_link.STL" />
+          filename="file://$(find robot_arm_6axis)/meshes/wrist_link.STL" />
+      </geometry>
+      <material
+        name="">
+        <color
+          rgba="0.792156862745098 0.819607843137255 0.933333333333333 1" />
+      </material>
+    </visual>
+    <collision>
+      <origin
+        xyz="0 0 0"
+        rpy="0 0 0" />
+      <geometry>
+        <mesh
+          filename="file://$(find robot_arm_6axis)/meshes/wrist_link.STL" />
       </geometry>
     </collision>
@@ -225,19 +225,19 @@
       <geometry>
         <mesh
-          filename="package://robot_arm_6axis/meshes/hand_link.STL" />
-      </geometry>
-      <material
-        name="">
-        <color
-          rgba="0.792156862745098 0.819607843137255 0.933333333333333 1" />
-      </material>
-    </visual>
-    <collision>
-      <origin
-        xyz="0 0 0"
-        rpy="0 0 0" />
-      <geometry>
-        <mesh
-          filename="package://robot_arm_6axis/meshes/hand_link.STL" />
+          filename="file://$(find robot_arm_6axis)/meshes/hand_link.STL" />
+      </geometry>
+      <material
+        name="">
+        <color
+          rgba="0.792156862745098 0.819607843137255 0.933333333333333 1" />
+      </material>
+    </visual>
+    <collision>
+      <origin
+        xyz="0 0 0"
+        rpy="0 0 0" />
+      <geometry>
+        <mesh
+          filename="file://$(find robot_arm_6axis)/meshes/hand_link.STL" />
       </geometry>
     </collision>
@@ -278,19 +278,19 @@
       <geometry>
         <mesh
-          filename="package://robot_arm_6axis/meshes/finger_link.STL" />
-      </geometry>
-      <material
-        name="">
-        <color
-          rgba="0.792156862745098 0.819607843137255 0.933333333333333 1" />
-      </material>
-    </visual>
-    <collision>
-      <origin
-        xyz="0 0 0"
-        rpy="0 0 0" />
-      <geometry>
-        <mesh
-          filename="package://robot_arm_6axis/meshes/finger_link.STL" />
+          filename="file://$(find robot_arm_6axis)/meshes/finger_link.STL" />
+      </geometry>
+      <material
+        name="">
+        <color
+          rgba="0.792156862745098 0.819607843137255 0.933333333333333 1" />
+      </material>
+    </visual>
+    <collision>
+      <origin
+        xyz="0 0 0"
+        rpy="0 0 0" />
+      <geometry>
+        <mesh
+          filename="file://$(find robot_arm_6axis)/meshes/finger_link.STL" />
       </geometry>
     </collision>
@@ -331,19 +331,19 @@
       <geometry>
         <mesh
-          filename="package://robot_arm_6axis/meshes/tip_link.STL" />
-      </geometry>
-      <material
-        name="">
-        <color
-          rgba="0.792156862745098 0.819607843137255 0.933333333333333 1" />
-      </material>
-    </visual>
-    <collision>
-      <origin
-        xyz="0 0 0"
-        rpy="0 0 0" />
-      <geometry>
-        <mesh
-          filename="package://robot_arm_6axis/meshes/tip_link.STL" />
+          filename="file://$(find robot_arm_6axis)/meshes/tip_link.STL" />
+      </geometry>
+      <material
+        name="">
+        <color
+          rgba="0.792156862745098 0.819607843137255 0.933333333333333 1" />
+      </material>
+    </visual>
+    <collision>
+      <origin
+        xyz="0 0 0"
+        rpy="0 0 0" />
+      <geometry>
+        <mesh
+          filename="file://$(find robot_arm_6axis)/meshes/tip_link.STL" />
       </geometry>
     </collision>
