Commit message: fixed packaging names

File: urdf/epsonvt6_core.xacro (robot description, xacro)
@@ -30,5 +30,5 @@
       <geometry>
         <mesh
-          filename="file://$(find robot_arm_6axis)/meshes/base_link.STL" /> <!-- package://robot_arm_6axis/meshes/base_link.STL"-->
+          filename="file://$(find epsonvt6_sim)/meshes/base_link.STL" /> <!-- package://epsonvt6_sim/meshes/base_link.STL"-->
       </geometry>
       <material
@@ -44,5 +44,5 @@
       <geometry>
         <mesh
-          filename="file://$(find robot_arm_6axis)/meshes/base_link.STL" />
+          filename="file://$(find epsonvt6_sim)/meshes/base_link.STL" />
       </geometry>
     </collision>
@@ -70,5 +70,5 @@
       <geometry>
         <mesh
-          filename="file://$(find robot_arm_6axis)/meshes/swivel_link.STL" />
+          filename="file://$(find epsonvt6_sim)/meshes/swivel_link.STL" />
       </geometry>
       <material
@@ -84,5 +84,5 @@
       <geometry>
         <mesh
-          filename="file://$(find robot_arm_6axis)/meshes/swivel_link.STL" />
+          filename="file://$(find epsonvt6_sim)/meshes/swivel_link.STL" />
       </geometry>
     </collision>
@@ -123,19 +123,19 @@
       <geometry>
         <mesh
-          filename="file://$(find robot_arm_6axis)/meshes/swivel_arm_link.STL" />
-      </geometry>
-      <material
-        name="">
-        <color
-          rgba="0.792156862745098 0.819607843137255 0.933333333333333 1" />
-      </material>
-    </visual>
-    <collision>
-      <origin
-        xyz="0 0 0"
-        rpy="0 0 0" />
-      <geometry>
-        <mesh
-          filename="file://$(find robot_arm_6axis)/meshes/swivel_arm_link.STL" />
+          filename="file://$(find epsonvt6_sim)/meshes/swivel_arm_link.STL" />
+      </geometry>
+      <material
+        name="">
+        <color
+          rgba="0.792156862745098 0.819607843137255 0.933333333333333 1" />
+      </material>
+    </visual>
+    <collision>
+      <origin
+        xyz="0 0 0"
+        rpy="0 0 0" />
+      <geometry>
+        <mesh
+          filename="file://$(find epsonvt6_sim)/meshes/swivel_arm_link.STL" />
       </geometry>
     </collision>
@@ -176,19 +176,19 @@
       <geometry>
         <mesh
-          filename="file://$(find robot_arm_6axis)/meshes/wrist_link.STL" />
-      </geometry>
-      <material
-        name="">
-        <color
-          rgba="0.792156862745098 0.819607843137255 0.933333333333333 1" />
-      </material>
-    </visual>
-    <collision>
-      <origin
-        xyz="0 0 0"
-        rpy="0 0 0" />
-      <geometry>
-        <mesh
-          filename="file://$(find robot_arm_6axis)/meshes/wrist_link.STL" />
+          filename="file://$(find epsonvt6_sim)/meshes/wrist_link.STL" />
+      </geometry>
+      <material
+        name="">
+        <color
+          rgba="0.792156862745098 0.819607843137255 0.933333333333333 1" />
+      </material>
+    </visual>
+    <collision>
+      <origin
+        xyz="0 0 0"
+        rpy="0 0 0" />
+      <geometry>
+        <mesh
+          filename="file://$(find epsonvt6_sim)/meshes/wrist_link.STL" />
       </geometry>
     </collision>
@@ -229,19 +229,19 @@
       <geometry>
         <mesh
-          filename="file://$(find robot_arm_6axis)/meshes/hand_link.STL" />
-      </geometry>
-      <material
-        name="">
-        <color
-          rgba="0.792156862745098 0.819607843137255 0.933333333333333 1" />
-      </material>
-    </visual>
-    <collision>
-      <origin
-        xyz="0 0 0"
-        rpy="0 0 0" />
-      <geometry>
-        <mesh
-          filename="file://$(find robot_arm_6axis)/meshes/hand_link.STL" />
+          filename="file://$(find epsonvt6_sim)/meshes/hand_link.STL" />
+      </geometry>
+      <material
+        name="">
+        <color
+          rgba="0.792156862745098 0.819607843137255 0.933333333333333 1" />
+      </material>
+    </visual>
+    <collision>
+      <origin
+        xyz="0 0 0"
+        rpy="0 0 0" />
+      <geometry>
+        <mesh
+          filename="file://$(find epsonvt6_sim)/meshes/hand_link.STL" />
       </geometry>
     </collision>
@@ -282,19 +282,19 @@
       <geometry>
         <mesh
-          filename="file://$(find robot_arm_6axis)/meshes/finger_link.STL" />
-      </geometry>
-      <material
-        name="">
-        <color
-          rgba="0.792156862745098 0.819607843137255 0.933333333333333 1" />
-      </material>
-    </visual>
-    <collision>
-      <origin
-        xyz="0 0 0"
-        rpy="0 0 0" />
-      <geometry>
-        <mesh
-          filename="file://$(find robot_arm_6axis)/meshes/finger_link.STL" />
+          filename="file://$(find epsonvt6_sim)/meshes/finger_link.STL" />
+      </geometry>
+      <material
+        name="">
+        <color
+          rgba="0.792156862745098 0.819607843137255 0.933333333333333 1" />
+      </material>
+    </visual>
+    <collision>
+      <origin
+        xyz="0 0 0"
+        rpy="0 0 0" />
+      <geometry>
+        <mesh
+          filename="file://$(find epsonvt6_sim)/meshes/finger_link.STL" />
       </geometry>
     </collision>
@@ -335,19 +335,19 @@
       <geometry>
         <mesh
-          filename="file://$(find robot_arm_6axis)/meshes/tip_link.STL" />
-      </geometry>
-      <material
-        name="">
-        <color
-          rgba="0.792156862745098 0.819607843137255 0.933333333333333 1" />
-      </material>
-    </visual>
-    <collision>
-      <origin
-        xyz="0 0 0"
-        rpy="0 0 0" />
-      <geometry>
-        <mesh
-          filename="file://$(find robot_arm_6axis)/meshes/tip_link.STL" />
+          filename="file://$(find epsonvt6_sim)/meshes/tip_link.STL" />
+      </geometry>
+      <material
+        name="">
+        <color
+          rgba="0.792156862745098 0.819607843137255 0.933333333333333 1" />
+      </material>
+    </visual>
+    <collision>
+      <origin
+        xyz="0 0 0"
+        rpy="0 0 0" />
+      <geometry>
+        <mesh
+          filename="file://$(find epsonvt6_sim)/meshes/tip_link.STL" />
       </geometry>
     </collision>

Commit message: configerd to work with the harvad repo

File: urdf/epsonvt6_core.xacro (robot description, xacro)
@@ -8,4 +8,12 @@
 -->
 <robot xmlns:xacro="http://www.ros.org/wiki/xacro">
+  <link name="world">
+     <origin xyz="0 0 0" rpy="0 0 0"/>
+  </link>
+  <joint name="world_joint" type="fixed">
+    <origin xyz="0 0 0.3" rpy="0 0 0"/>
+    <parent link="world"/>
+    <child link="base_link"/>
+  </joint>
   <link
     name="base_link">
